Commit message: Fixed URDF not being able to reference the mesh files

File: urdf/sjtu_drone.urdf (robot description, URDF)
Before this commit: robot sjtu_drone, 1 links, 0 joints
Links:
- link base_link: geometry collision mesh filename=file://meshes/quadrotor_4.stl; visual mesh filename=file://meshes/quadrotor_4.dae
